File: arcade-game.brd (EAGLE design)
At the start: 235.1 x 197.2 mm, 7 parts, among them U1 ARDUINO-UNO-R3-SHIELD, U2 ARDUINO-UNO-R3-SHIELD, U3 LCD-16X2-I2CSUNFOUNDER-IIC, U4 LCD-16X2-I2CSUNFOUNDER-IIC, U5 ARDUINO-UNO-R3-SHIELD

Commit message: Add files via upload
Parts:
- removed S1, S2: SWITCH_MOMENTARY, Tinkercad:SWITCH-MOMENTARY-PTH-6.5MM
- U1: value ARDUINO-UNO-R3-SHIELD -> IR-RECEIVERTSOP48; device Tinkercad:ARDUINO-UNO-R3-SHIELD -> Tinkercad:TSOP48
- moved U1 35.3 mm to (50.7, 118.8), turned to 180 degrees
Connections:
- removed net U1_D2: S1.1, S1.2, U1.D2
- removed net U1_D3: S2.1, S2.2, U1.D3
- removed net U1_D8: U1.D8, U5.D2
- removed net U1_D9: U1.D9, U5.D3
- removed net U1_GND: S1.3, S1.4, S2.3, S2.4, U1.GND@0, U1.GND@1, U1.GND@2, U2.GND@0, U2.GND@1, U2.GND@2, U3.1, U4.1, U5.GND@0, U5.GND@1, U5.GND@2
- new net U2_GND: U1.2, U2.GND@0, U2.GND@1, U2.GND@2, U3.1, U4.1, U5.GND@0, U5.GND@1, U5.GND@2
- new net U5_5V: U1.3, U5.5V
- new net U5_D11: U1.1, U5.D11
Changed lines of the file:
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@@
 </autorouter>
 <elements>
-<element name="S2" library="Tinkercad" library_urn="urn:adsk.eagle:library:30890021" package="SWITCH-MOMENTARY-PTH-6.5MM" package3d_urn="urn:adsk.eagle:package:32246662/3" value="SWITCH_MOMENTARY" x="87.135" y="22.9098" rot="R90" smashed="yes"/>
-<element name="S1" library="Tinkercad" library_urn="urn:adsk.eagle:library:30890021" package="SWITCH-MOMENTARY-PTH-6.5MM" package3d_urn="urn:adsk.eagle:package:32246662/3" value="SWITCH_MOMENTARY" x="31.255" y="22.9098" rot="R90" smashed="yes"/>
-<element name="U1" library="Tinkercad" library_urn="urn:adsk.eagle:library:30890021" package="ARDUINO-UNO-R3-SHIELD" package3d_urn="urn:adsk.eagle:package:32092383/4" value="ARDUINO-UNO-R3-SHIELD" x="56.1673" y="83.8847" rot="R270" smashed="yes"/>
-<element name="U5" library="Tinkercad" library_urn="urn:adsk.eagle:library:30890021" package="ARDUINO-UNO-R3-SHIELD" package3d_urn="urn:adsk.eagle:package:32092383/4" value="ARDUINO-UNO-R3-SHIELD" x="47.885" y="154.7063" rot="R270" smashed="yes"/>
 <element name="U4" library="Tinkercad" library_urn="urn:adsk.eagle:library:30890021" package="LCD-I2C" package3d_urn="urn:adsk.eagle:package:35699708/2" value="LCD-16X2-I2CSUNFOUNDER-IIC" x="177.819" y="158.5195" smashed="yes"/>
 <element name="U3" library="Tinkercad" library_urn="urn:adsk.eagle:library:30890021" package="LCD-I2C" package3d_urn="urn:adsk.eagle:package:35699708/2" value="LCD-16X2-I2CSUNFOUNDER-IIC" x="177.8092" y="189.6843" smashed="yes"/>
 <element name="U2" library="Tinkercad" library_urn="urn:adsk.eagle:library:30890021" package="ARDUINO-UNO-R3-SHIELD" package3d_urn="urn:adsk.eagle:package:32092383/4" value="ARDUINO-UNO-R3-SHIELD" x="200.5426" y="29.845" rot="R270" smashed="yes"/>
+<element name="U5" library="Tinkercad" library_urn="urn:adsk.eagle:library:30890021" package="ARDUINO-UNO-R3-SHIELD" package3d_urn="urn:adsk.eagle:package:32092383/4" value="ARDUINO-UNO-R3-SHIELD" x="47.885" y="154.7063" rot="R270" smashed="yes"/>
+<element name="U1" library="Tinkercad" library_urn="urn:adsk.eagle:library:30890021" package="TSOP48" package3d_urn="urn:adsk.eagle:package:32501402/2" value="IR-RECEIVERTSOP48" x="50.7034" y="118.7659" rot="R180" smashed="yes"/>
 </elements>
 <signals>
-<signal name="U1_GND">
-<contactref element="S1" pad="4"/>
-<contactref element="S2" pad="3"/>
-<contactref element="S1" pad="3"/>
-<contactref element="U1" pad="GND@0"/>
-<contactref element="U1" pad="GND@1"/>
-<contactref element="U1" pad="GND@2"/>
-<contactref element="S2" pad="4"/>
+<signal name="U2_GND">
 <contactref element="U2" pad="GND@0"/>
 <contactref element="U2" pad="GND@1"/>
@@
 <contactref element="U4" pad="1"/>
 <contactref element="U3" pad="1"/>
+<contactref element="U1" pad="2"/>
 <contactref element="U5" pad="GND@0"/>
 <contactref element="U5" pad="GND@1"/>
@@
 <wire x1="203.0826" y1="5.715" x2="205.6226" y2="5.715" width="0" layer="19" extent="1-1"/>
 <wire x1="203.0826" y1="5.715" x2="189.1126" y2="53.975" width="0" layer="19" extent="1-1"/>
-<wire x1="89.3956" y1="26.161" x2="189.1126" y2="53.975" width="0" layer="19" extent="1-1"/>
-<wire x1="89.3956" y1="19.6586" x2="89.3956" y2="26.161" width="0" layer="19" extent="1-1"/>
-<wire x1="61.2473" y1="59.7547" x2="89.3956" y2="26.161" width="0" layer="19" extent="1-1"/>
-<wire x1="58.7073" y1="59.7547" x2="61.2473" y2="59.7547" width="0" layer="19" extent="1-1"/>
-<wire x1="33.5156" y1="26.161" x2="58.7073" y2="59.7547" width="0" layer="19" extent="1-1"/>
-<wire x1="33.5156" y1="26.161" x2="33.5156" y2="19.6586" width="0" layer="19" extent="1-1"/>
-<wire x1="58.7073" y1="59.7547" x2="44.7373" y2="108.0147" width="0" layer="19" extent="1-1"/>
-<wire x1="44.7373" y1="108.0147" x2="50.425" y2="130.5763" width="0" layer="19" extent="1-1"/>
-<wire x1="50.425" y1="130.5763" x2="52.965" y2="130.5763" width="0" layer="19" extent="1-1"/>
-<wire x1="50.425" y1="130.5763" x2="36.455" y2="178.8363" width="0" layer="19" extent="1-1"/>
 <wire x1="189.1126" y1="53.975" x2="158.769" y2="153.4395" width="0" layer="19" extent="1-1"/>
 <wire x1="158.769" y1="153.4395" x2="158.7592" y2="184.6043" width="0" layer="19" extent="1-1"/>
-</signal>
-<signal name="U1_D3">
-<contactref element="S2" pad="2"/>
-<contactref element="U1" pad="D3"/>
-<contactref element="S2" pad="1"/>
-<wire x1="84.8744" y1="26.161" x2="84.8744" y2="19.6586" width="0" layer="19" extent="1-1"/>
-<wire x1="84.8744" y1="26.161" x2="73.9473" y2="108.0147" width="0" layer="19" extent="1-1"/>
-</signal>
-<signal name="U1_D2">
-<contactref element="S1" pad="2"/>
-<contactref element="U1" pad="D2"/>
-<contactref element="S1" pad="1"/>
-<wire x1="28.9944" y1="26.161" x2="28.9944" y2="19.6586" width="0" layer="19" extent="1-1"/>
-<wire x1="28.9944" y1="26.161" x2="76.4873" y2="108.0147" width="0" layer="19" extent="1-1"/>
-</signal>
-<signal name="U1_D9">
-<contactref element="U1" pad="D9"/>
-<contactref element="U5" pad="D3"/>
-<wire x1="57.4373" y1="108.0147" x2="65.665" y2="178.8363" width="0" layer="19" extent="1-1"/>
-</signal>
-<signal name="U1_D8">
-<contactref element="U1" pad="D8"/>
-<contactref element="U5" pad="D2"/>
-<wire x1="59.9773" y1="108.0147" x2="68.205" y2="178.8363" width="0" layer="19" extent="1-1"/>
-</signal>
-<signal name="U5_TX">
-<contactref element="U5" pad="TX"/>
-<contactref element="U2" pad="RX"/>
-<wire x1="70.745" y1="178.8363" x2="225.9426" y2="53.975" width="0" layer="19" extent="1-1"/>
+<wire x1="158.769" y1="153.4395" x2="52.965" y2="130.5763" width="0" layer="19" extent="1-1"/>
+<wire x1="50.425" y1="130.5763" x2="52.965" y2="130.5763" width="0" layer="19" extent="1-1"/>
+<wire x1="50.7034" y1="118.7659" x2="50.425" y2="130.5763" width="0" layer="19" extent="1-1"/>
+<wire x1="50.425" y1="130.5763" x2="36.455" y2="178.8363" width="0" layer="19" extent="1-1"/>
 </signal>
 <signal name="U2_A5">
@@
 <wire x1="200.5426" y1="5.715" x2="158.769" y2="150.8995" width="0" layer="19" extent="1-1"/>
 </signal>
+<signal name="U5_TX">
+<contactref element="U5" pad="TX"/>
+<contactref element="U2" pad="RX"/>
+<wire x1="70.745" y1="178.8363" x2="225.9426" y2="53.975" width="0" layer="19" extent="1-1"/>
+</signal>
+<signal name="U5_D11">
+<contactref element="U1" pad="1"/>
+<contactref element="U5" pad="D11"/>
+<wire x1="53.2434" y1="118.7659" x2="44.075" y2="178.8363" width="0" layer="19" extent="1-1"/>
+</signal>
+<signal name="U5_5V">
+<contactref element="U1" pad="3"/>
+<contactref element="U5" pad="5V"/>
+<wire x1="48.1634" y1="118.7659" x2="47.885" y2="130.5763" width="0" layer="19" extent="1-1"/>
+</signal>
 </signals>
